Commit message: Complete tutorial Exercise 3.1: Workcell XACRO

File: myworkcell_support/urdf/workcell.xacro (robot description, xacro)
@@ -1,14 +1,21 @@
 <?xml version="1.0"?>
 <robot name="myworkcell" xmlns:xacro="http://www.ros.org/wiki/xacro">
+    <xacro:include filename="$(find ur_description)/urdf/ur5.urdf.xacro" />
+    <xacro:ur5_robot prefix="" joint_limited="true"/>
+    <joint name="table_to_robot" type="fixed">
+        <parent link="table"/>
+        <child link="base_link"/>
+        <origin xyz="0 0 0" rpy="0 0 0"/>
+    </joint>
     <link name="world"/>
     <link name="table">
         <visual>
           <geometry>
-            <box size="0.6 0.6 2.0"/>
+            <box size="0.6 0.6 0.05"/>
           </geometry>
         </visual>
         <collision>
           <geometry>
-            <box size="0.6 0.6 2.0"/>
+            <box size="0.6 0.6 0.05"/>
           </geometry>
         </collision>

Commit message: Add memo/E4-0_Motion_Planning_C++.md

File: myworkcell_support/urdf/workcell.xacro (robot description, xacro)
@@ -30,5 +30,5 @@
         <parent link="world"/>
         <child link="camera_frame"/>
-        <origin xyz="0 0 1.0" rpy="0 1.571 0"/>
+        <origin xyz="0 0 1.0" rpy="0 3.14159 0"/>
     </joint>
 </robot>
